File: KEA_Demo.sch (KiCad schematic (older format))
At the start: 6 parts, among them P1 PWR

Commit message: Finished Schematic
Parts:
- added D?: 1N4001, symbol D
- added P?: JTAG, symbol CONN_01X05
- added P?: SPI, symbol CONN_01X06
- added P? (x2): I2C, symbol CONN_01X04
Connections:
- net +3V3: now also P?.1 (P1), P?.4 (P4), P?.4 (P4), P?.6 (P6)
- net GND: now also P?.1 (P1), P?.1 (P1), P?.1 (P1), P?.5 (P5)
- net nReset: now reaches U?.1 (PTA5)
- net nReset: now also P?.2 (P2)
- net SPI0_SCK: now reaches U?.10 (PTB2)
- net SPI0_SCK: now also P?.2 (P2)
- net UART0_TX: now reaches U?.11 (PTB1)
- net UART0_TX: now also P?.3 (P3)
- net UART0_RX: now reaches U?.12 (PTB0)
- net UART0_RX: now also P?.2 (P2)
- net FTM0_CH1: now reaches U?.15 (PTA1)
- net FTM0_CH0: now reaches U?.16 (PTA0)
- net FTM0_CH0: now also P?.4 (P4)
- net SDIO: now reaches U?.2 (PTA4)
- net SDIO: now also P?.3 (P3)
- net I2C0_SCL: now reaches U?.5 (PTB7)
- net I2C0_SCL: now also P?.3 (P3)
- net I2C0_SDA: now reaches U?.6 (PTB6)
- net I2C0_SDA: now also P?.2 (P2)
- net SPI0_PCS: now reaches U?.7 (PTB5)
- net SPI0_PCS: now also P?.5 (P5)
- net SPI0_MISO: now reaches U?.8 (PTB4)
- net SPI0_MISO: now also P?.3 (P3)
- net SPI0_MOSI: now reaches U?.9 (PTB3)
- net SPI0_MOSI: now also P?.4 (P4)
- net at C?.1, U?.3 (VI): now also D?.1 (K); no longer P1.1 (P1)
- new net: D?.2 (A), P1.1 (P1)
Other:
- moved on the sheet: P1
